Commit message: three camer implementation

File: interbotix_xsarm_descriptions/urdf/wx250s.urdf.xacro (robot description, xacro)
@@ -391,5 +391,5 @@
       <child link="$(arg robot_name)/frypan_link"/>
     </joint>
-    <xacro:if value="$(arg show_frypan)">
+    <!-- <xacro:if value="$(arg show_frypan)">
       <link name="$(arg robot_name)/frypan_link">
         <visual>
@@ -404,4 +404,26 @@
           <geometry>
             <mesh filename="package://interbotix_xsarm_descriptions/meshes/wx250s_meshes/wx250s_12_frypan.stl" scale="0.001 0.001 0.001"/>
+          </geometry>
+        </collision>
+        <inertial>
+          <origin rpy="0 0 ${pi/2}" xyz="0.0096870000 0.0000008177 0.0049620000"/>
+          <mass value="0.5" />
+          <inertia ixx="0.0000074125" iyy="0.0000284300" izz="0.0000286000" ixy="-0.0000000008" ixz="-0.0000000006" iyz="-0.0000013889" />
+        </inertial>
+      </link>
+    </xacro:if> -->
+    <xacro:if value="$(arg show_frypan)">
+      <link name="$(arg robot_name)/frypan_link">
+        <visual>
+          <origin rpy="${pi} ${pi} ${pi/2}" xyz="0.095 0 -0.0285"/>
+          <geometry>
+            <mesh filename="package://interbotix_xsarm_descriptions/meshes/wx250s_meshes/wx250s_12_frypan.stl" scale="0.00075 0.00075 0.00075"/>
+          </geometry>
+          <material name="interbotix_black"/>
+        </visual>
+        <collision>
+          <origin rpy="${pi} ${pi} ${pi/2}" xyz="0.095 0 -0.0285"/>
+          <geometry>
+            <mesh filename="package://interbotix_xsarm_descriptions/meshes/wx250s_meshes/wx250s_12_frypan.stl" scale="0.00075 0.00075 0.00075"/>
           </geometry>
         </collision>
